File: monolith_kicad/_saved_monolith.sch (KiCad schematic (older format))
At the start: 9 parts

Commit message: updated pcb
Made smaller + added name/rev/date/etc
Connections:
- net at U?.1 (REST): now also SW?.1
- net at U?.15 (RXD): now also P?.2 (P2)
- net at U?.16 (TXD): now also P?.3 (P3)
- net at BT?.2 (-), P?.1 (P1), P?.2 (P2)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: now also P?.6 (P6)
- net at SW?.2: now also SW?.1
Other:
- moved on the sheet: SW?
Changed lines of the file:
@@
 	3250 4550 6850 4550
 Wire Wire Line
-	6700 4550 6700 3800
+	6700 3800 6700 5300
 Connection ~ 4250 4550
 Wire Wire Line
@@
 	6700 3500 7050 3500
 Wire Wire Line
-	7050 3500 7050 4750
+	7050 1850 7050 4750
 Wire Wire Line
 	7050 4750 4400 4750
@@
 L SW_DIP_x01 SW?
 U 1 1 5997975E
-P 6150 5400
-F 0 "SW?" H 6150 5550 50  0000 C CNN
-F 1 "SW_DIP_x01" H 6150 5250 50  0000 C CNN
-F 2 "" H 6150 5400 50  0000 C CNN
-F 3 "" H 6150 5400 50  0000 C CNN
-	1    6150 5400
+P 5050 1850
+F 0 "SW?" H 5050 2000 50  0000 C CNN
+F 1 "SW_DIP_x01" H 5050 1700 50  0000 C CNN
+F 2 "" H 5050 1850 50  0000 C CNN
+F 3 "" H 5050 1850 50  0000 C CNN
+	1    5050 1850
 	1    0    0    -1
 $EndComp
@@
 L SW_DIP_x01 SW?
 U 1 1 59979863
-P 6150 5750
-F 0 "SW?" H 6150 5900 50  0000 C CNN
-F 1 "SW_DIP_x01" H 6150 5600 50  0000 C CNN
-F 2 "" H 6150 5750 50  0000 C CNN
-F 3 "" H 6150 5750 50  0000 C CNN
-	1    6150 5750
+P 6100 1850
+F 0 "SW?" H 6100 2000 50  0000 C CNN
+F 1 "SW_DIP_x01" H 6100 1700 50  0000 C CNN
+F 2 "" H 6100 1850 50  0000 C CNN
+F 3 "" H 6100 1850 50  0000 C CNN
+	1    6100 1850
 	1    0    0    -1
 $EndComp
+Wire Wire Line
+	6700 3200 7250 3200
+Wire Wire Line
+	7250 3200 7250 4900
+Wire Wire Line
+	7250 4900 7750 4900
+Wire Wire Line
+	7750 5000 7350 5000
+Wire Wire Line
+	7350 5000 7350 3100
+Wire Wire Line
+	7350 3100 6700 3100
+Wire Wire Line
+	6700 5300 7750 5300
+Wire Wire Line
+	4900 3100 4500 3100
+Wire Wire Line
+	4500 3100 4500 1850
+Wire Wire Line
+	4500 1850 4750 1850
+Wire Wire Line
+	5350 1850 5800 1850
+Wire Wire Line
+	7050 1850 6350 1850
+Connection ~ 7050 3500
 $EndSCHEMATC
