File: monolith_kicad/monolith.kicad_pcb (KiCad board)
At the start: 2 copper layers, 55.9 x 33 mm, 9 parts

Commit message: updated pcb
Made smaller + added name/rev/date/etc
Parts:
- AMS1117 3.3V: renamed from REF**; value SOT-223 -> -|3.3v|5v
- moved REF** 6.99 mm to (155.6, 90.2)
- moved   5.72 mm to (145.4, 90.2)
- moved ? 5.08 mm to (133.3, 90.2)
- moved AMS1117 3.3V 2.84 mm to (129.5, 78.1)
- renumbered REF** to ?
Routing:
- net (no net): track 491.0 -> 494.0 mm
Other:
- board size 55.9 x 33 mm -> 44.5 x 33 mm
- board text added: "BOT"
- board text added: "GND 5V"
- board text added: "GND D 5V"
- board text added: "Monolith rev 1.0 Aug 2017 Dominick Anatala"
- board text added: "TOP"
- board text removed: "- +"
- board text removed: "- D +"

Commit message: continued update pcb + housing
Parts:
-  : renamed from REF**
- AMS1117 3.3V: value -|3.3v|5v -> GND|3.3V|5V
Routing:
- net (no net): track 494.0 -> 495.9 mm
Other:
- board text added: "3.3V TX RX GND"
- board text added: "VCC GND SCL SDA AD0 INT"
- board text removed: "GND RX TX 3.3V"
- board text removed: "VCC GND SCL SDA INT"
Changed lines of the file:
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@@
     (thickness 1.6)
     (drawings 19)
-    (tracks 201)
+    (tracks 203)
     (zones 0)
     (modules 9)
@@
     (descr "Through hole straight socket strip, 1x02, 2.54mm pitch, single row")
     (tags "Through hole socket strip THT 1x02 2.54mm single row")
-    (fp_text reference REF** (at 0 -2.33 90) (layer F.SilkS)
+    (fp_text reference " " (at 0 -2.33 90) (layer F.SilkS)
       (effects (font (size 1 1) (thickness 0.15)))
     )
@@
     (tags "CMS SOT")
     (attr smd)
-    (fp_text reference "AMS1117 3.3V" (at 0 4.5 180) (layer B.SilkS)
+    (fp_text reference "AMS1117 3.3V" (at 0.635 4.445 180) (layer B.SilkS)
       (effects (font (size 1 1) (thickness 0.15)) (justify mirror))
     )
-    (fp_text value -|3.3v|5v (at -5.0292 -0.1778 270) (layer B.SilkS)
-      (effects (font (size 0.8 0.8) (thickness 0.15)) (justify mirror))
+    (fp_text value GND|3.3V|5V (at -5.1054 0.4699 270) (layer B.SilkS)
+      (effects (font (size 0.7 0.7) (thickness 0.12)) (justify mirror))
     )
     (fp_text user %R (at 0 0 450) (layer B.Fab)
@@
     )
   )
+  (gr_text "3.3V TX RX GND" (at 154.20086 77.72908 90) (layer F.SilkS)
+    (effects (font (size 0.9 0.9) (thickness 0.2)))
+  )
   (dimension 44.45 (width 0.3) (layer F.Fab)
     (gr_text "44.450 mm" (at 144.145 57.705) (layer F.Fab)
@@
     (effects (font (size 1.5 1.5) (thickness 0.3)))
   )
-  (gr_text "Monolith rev 1.0\nAug 2017\nDominick Anatala" (at 160.02 76.835 90) (layer F.SilkS)
+  (gr_text "Monolith\nrev 1.0 Aug 2017\nDominick Anatala" (at 160.02 78.105 90) (layer F.SilkS)
     (effects (font (size 1.5 1.5) (thickness 0.3)))
   )
@@
   )
   (gr_circle (center 125.095 90.805) (end 125.095 92.305) (layer Edge.Cuts) (width 0.15))
-  (gr_text "GND RX TX 3.3V" (at 149.225 77.47 270) (layer F.SilkS)
-    (effects (font (size 0.9 0.9) (thickness 0.2)))
-  )
-  (gr_text "VCC GND SCL SDA                INT" (at 139.065 66.04) (layer F.SilkS)
+  (gr_text "VCC GND SCL SDA          AD0  INT" (at 139.065 66.04) (layer F.SilkS)
     (effects (font (size 0.8 0.7) (thickness 0.175)))
   )
@@
   (gr_circle (center 163.195 64.135) (end 163.195 65.635) (layer Edge.Cuts) (width 0.15))
   (gr_line (start 121.92 60.96) (end 121.92 93.98) (angle 90) (layer Edge.Cuts) (width 0.15))
+  (segment (start 144.78 66.04) (end 145.415 65.405) (width 0.25) (layer F.Cu) (net 0))
+  (segment (start 145.415 65.405) (end 145.415 64.135) (width 0.25) (layer F.Cu) (net 0) (status 800000))
   (segment (start 150.495 83.82) (end 148.59 85.725) (width 0.25) (layer F.Cu) (net 0))
   (segment (start 148.59 85.725) (end 146.685 87.63) (width 0.25) (layer F.Cu) (net 0))
@@
   (segment (start 135.89 80.645) (end 133.985 80.645) (width 0.25) (layer B.Cu) (net 0))
   (segment (start 150.495 85.09) (end 151.13 85.09) (width 0.25) (layer B.Cu) (net 0))
-  (segment (start 151.13 85.09) (end 156.21 85.09) (width 0.5) (layer B.Cu) (net 0))
-  (segment (start 156.21 85.09) (end 157.48 85.09) (width 0.5) (layer B.Cu) (net 0))
+  (segment (start 151.13 85.09) (end 155.575 85.09) (width 0.5) (layer B.Cu) (net 0))
+  (segment (start 155.575 85.09) (end 157.48 85.09) (width 0.5) (layer B.Cu) (net 0))
   (segment (start 158.115 85.725) (end 158.115 90.17) (width 0.5) (layer B.Cu) (net 0))
   (segment (start 157.48 85.09) (end 158.115 85.725) (width 0.5) (layer B.Cu) (net 0))
@@
   (segment (start 129.54 83.185) (end 133.35 83.185) (width 0.25) (layer F.Cu) (net 0))
   (segment (start 153.035 71.12) (end 153.67 71.12) (width 0.25) (layer B.Cu) (net 0))
-  (segment (start 156.21 73.66) (end 156.21 74.295) (width 0.25) (layer B.Cu) (net 0))
-  (segment (start 153.67 71.12) (end 156.21 73.66) (width 0.25) (layer B.Cu) (net 0))
+  (segment (start 153.67 71.12) (end 155.575 73.025) (width 0.25) (layer B.Cu) (net 0))
+  (segment (start 153.67 71.12) (end 153.67 71.12) (width 0.25) (layer B.Cu) (net 0))
   (segment (start 148.59 69.215) (end 150.495 71.12) (width 0.25) (layer F.Cu) (net 0))
   (segment (start 130.175 65.405) (end 131.445 66.675) (width 0.25) (layer F.Cu) (net 0))
@@
   (segment (start 146.05 66.675) (end 148.59 69.215) (width 0.25) (layer F.Cu) (net 0))
   (segment (start 145.415 66.675) (end 146.05 66.675) (width 0.25) (layer F.Cu) (net 0))
-  (segment (start 156.21 74.295) (end 156.21 85.09) (width 0.25) (layer B.Cu) (net 0))
+  (segment (start 155.575 73.025) (end 155.575 85.09) (width 0.25) (layer B.Cu) (net 0))
   (segment (start 150.495 71.12) (end 153.035 71.12) (width 0.25) (layer B.Cu) (net 0))
   (via (at 150.495 71.12) (size 0.6) (drill 0.4) (layers F.Cu B.Cu) (net 0))

Commit message: lots of updates since github desktop glitched out
updated pcb to v1.0 and am waiting for it to come back

updated case design to mostly 1.0

continued work on seperate controller using an esp8266

added basic BOM using mostly just components from amazon so anyone can easily buy the components needed to build this
Parts:
- added ?: BAT, Socket_Strips:Socket_Strip_Straight_1x01_Pitch2.54mm, F.Cu at (128.3, 88.9)
- added ?: 0.1 uF, Capacitors_SMD:C_0805_HandSoldering, B.Cu at (135.9, 76.8)
- added ?: , ESP8266:logo_large_8mm, F.Cu at (154.3, 67.3)
- moved AMS1117 3.3V 1.90 mm to (127.6, 78.1)
Connections:
-   pad 1: (no net) -> GND (x2)
- ? pad 2: (no net) -> GND
- ? pad 1: (no net) -> GND
- AMS1117 3.3V pad 1: (no net) -> GND
- ESP12 pad 9: (no net) -> GND
Routing:
- net GND: track 0.00 -> 106.3 mm, vias 0 -> 1
- net (no net): track 495.9 -> 401.9 mm, vias 13 -> 12
- added copper zone on B.Cu, net GND
- added copper zone on F.Cu, net GND
Other:
- board text added: "Monolith rev 1.0 Sep 2017 Dominick Anatala"
- board text removed: "Monolith rev 1.0 Aug 2017 Dominick Anatala"
