File: monolith_kicad/monolith.sch (KiCad schematic (older format))
At the start: 7 parts

Commit message: updated pcb
Made smaller + added name/rev/date/etc
Parts:
- added SW? (x2): SW_DIP_x01, symbol SW_DIP_x01
Connections:
- net at U?.15 (RXD): now also P?.2 (P2)
- net at U?.16 (TXD): now also P?.3 (P3)
- net at BT?.2 (-), P?.1 (P1), P?.2 (P2)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: now also P?.6 (P6)
Changed lines of the file:
@@
 LIBS:ESP8266
 LIBS:mpu-6050
+LIBS:switches
 LIBS:monolith-cache
 EELAYER 25 0
@@
 	3250 4550 6850 4550
 Wire Wire Line
-	6700 4550 6700 3800
+	6700 3800 6700 5300
 Connection ~ 4250 4550
 Wire Wire Line
@@
 	4550 3750 4750 3750
 Connection ~ 4750 3800
+$Comp
+L SW_DIP_x01 SW?
+U 1 1 5997975E
+P 6150 5400
+F 0 "SW?" H 6150 5550 50  0000 C CNN
+F 1 "SW_DIP_x01" H 6150 5250 50  0000 C CNN
+F 2 "" H 6150 5400 50  0000 C CNN
+F 3 "" H 6150 5400 50  0000 C CNN
+	1    6150 5400
+	1    0    0    -1
+$EndComp
+$Comp
+L SW_DIP_x01 SW?
+U 1 1 59979863
+P 6150 5750
+F 0 "SW?" H 6150 5900 50  0000 C CNN
+F 1 "SW_DIP_x01" H 6150 5600 50  0000 C CNN
+F 2 "" H 6150 5750 50  0000 C CNN
+F 3 "" H 6150 5750 50  0000 C CNN
+	1    6150 5750
+	1    0    0    -1
+$EndComp
+Wire Wire Line
+	6700 3200 7250 3200
+Wire Wire Line
+	7250 3200 7250 4900
+Wire Wire Line
+	7250 4900 7750 4900
+Wire Wire Line
+	7750 5000 7350 5000
+Wire Wire Line
+	7350 5000 7350 3100
+Wire Wire Line
+	7350 3100 6700 3100
+Wire Wire Line
+	6700 5300 7750 5300
 $EndSCHEMATC

Commit message: continued update pcb + housing
Connections:
- net at U?.1 (REST): now also SW?.1
- net at SW?.2: now also SW?.1
Other:
- moved on the sheet: SW?
Changed lines of the file:
@@
 	6700 3500 7050 3500
 Wire Wire Line
-	7050 3500 7050 4750
+	7050 1850 7050 4750
 Wire Wire Line
 	7050 4750 4400 4750
@@
 L SW_DIP_x01 SW?
 U 1 1 5997975E
-P 6150 5400
-F 0 "SW?" H 6150 5550 50  0000 C CNN
-F 1 "SW_DIP_x01" H 6150 5250 50  0000 C CNN
-F 2 "" H 6150 5400 50  0000 C CNN
-F 3 "" H 6150 5400 50  0000 C CNN
-	1    6150 5400
+P 5050 1850
+F 0 "SW?" H 5050 2000 50  0000 C CNN
+F 1 "SW_DIP_x01" H 5050 1700 50  0000 C CNN
+F 2 "" H 5050 1850 50  0000 C CNN
+F 3 "" H 5050 1850 50  0000 C CNN
+	1    5050 1850
 	1    0    0    -1
 $EndComp
@@
 L SW_DIP_x01 SW?
 U 1 1 59979863
-P 6150 5750
-F 0 "SW?" H 6150 5900 50  0000 C CNN
-F 1 "SW_DIP_x01" H 6150 5600 50  0000 C CNN
-F 2 "" H 6150 5750 50  0000 C CNN
-F 3 "" H 6150 5750 50  0000 C CNN
-	1    6150 5750
+P 6100 1850
+F 0 "SW?" H 6100 2000 50  0000 C CNN
+F 1 "SW_DIP_x01" H 6100 1700 50  0000 C CNN
+F 2 "" H 6100 1850 50  0000 C CNN
+F 3 "" H 6100 1850 50  0000 C CNN
+	1    6100 1850
 	1    0    0    -1
 $EndComp
@@
 Wire Wire Line
 	6700 5300 7750 5300
+Wire Wire Line
+	4900 3100 4500 3100
+Wire Wire Line
+	4500 3100 4500 1850
+Wire Wire Line
+	4500 1850 4750 1850
+Wire Wire Line
+	5350 1850 5800 1850
+Wire Wire Line
+	7050 1850 6350 1850
+Connection ~ 7050 3500
 $EndSCHEMATC

Commit message: lots of updates since github desktop glitched out
updated pcb to v1.0 and am waiting for it to come back

updated case design to mostly 1.0

continued work on seperate controller using an esp8266

added basic BOM using mostly just components from amazon so anyone can easily buy the components needed to build this
Parts:
- added 100k, R?: R, symbol R
- gave numbers to parts that had none: 9
Connections:
- net at U2.2 (ADC): now also R?.2
- net GND: now reaches BT1.2 (-), P1.1 (P1), P2.2 (P2), P3.6 (P6), P4.2 (P2), U1.1 (GND), U2.9 (GND)
- net GND: now also SW1.2, SW2.1
- new net: 100k.1, R?.1
- new net 3.7vBAT: 100k.2
Changed lines of the file:
@@
 $EndDescr
 $Comp
-L CONN_01X06 P?
+L CONN_01X06 P4
 U 1 1 59912CF2
 P 8150 2850
-F 0 "P?" H 8150 3200 50  0000 C CNN
+F 0 "P4" H 8150 3200 50  0000 C CNN
 F 1 "L298N" H 8150 2500 50  0000 C CNN
 F 2 "" H 8150 2850 50  0000 C CNN
@@
 $EndComp
 $Comp
-L Battery BT?
+L Battery BT1
 U 1 1 5991316B
 P 3250 4350
-F 0 "BT?" H 3350 4450 50  0000 L CNN
+F 0 "BT1" H 3350 4450 50  0000 L CNN
 F 1 "Battery" H 3350 4350 50  0000 L CNN
 F 2 "" V 3250 4410 50  0000 C CNN
@@
 $EndComp
 $Comp
-L LD1117S33TR U?
+L LD1117S33TR U1
 U 1 1 59913256
 P 4250 3950
-F 0 "U?" H 4250 4200 50  0000 C CNN
+F 0 "U1" H 4250 4200 50  0000 C CNN
 F 1 "LD1117S33TR" H 4250 4150 50  0000 C CNN
 F 2 "SOT-223" H 4250 4050 50  0000 C CNN
@@
 VCC\nGND\n1A\n2A\n3B\n4B
 $Comp
-L ESP-12E U?
+L ESP-12E U2
 U 1 1 59912C8C
 P 5800 3400
-F 0 "U?" H 5800 3300 50  0000 C CNN
+F 0 "U2" H 5800 3300 50  0000 C CNN
 F 1 "ESP-12E" H 5800 3500 50  0000 C CNN
 F 2 "" H 5800 3400 50  0001 C CNN
@@
 	7500 2800 7950 2800
 $Comp
-L CONN_01X03 P?
+L CONN_01X03 P1
 U 1 1 59914799
 P 3100 3300
-F 0 "P?" H 3100 3500 50  0000 C CNN
+F 0 "P1" H 3100 3500 50  0000 C CNN
 F 1 "WS2812" V 3200 3300 50  0000 C CNN
 F 2 "" H 3100 3300 50  0000 C CNN
@@
 Wire Wire Line
 	3300 3400 3700 3400
-Wire Wire Line
-	3700 3400 3700 4550
 Connection ~ 3700 4550
 $Comp
-L CONN_01X08 P?
+L CONN_01X08 P2
 U 1 1 5991E759
 P 4750 5600
-F 0 "P?" H 4750 6050 50  0000 C CNN
+F 0 "P2" H 4750 6050 50  0000 C CNN
 F 1 "MPU6050" H 4750 5150 50  0000 C CNN
 F 2 "" H 4750 5600 50  0000 C CNN
@@
 	7500 3700 7500 2800
 $Comp
-L CONN_01X06 P?
+L CONN_01X06 P3
 U 1 1 59967D01
 P 7950 5050
-F 0 "P?" H 7950 5400 50  0000 C CNN
+F 0 "P3" H 7950 5400 50  0000 C CNN
 F 1 "FTDI" H 7950 4650 50  0000 C CNN
 F 2 "" H 7950 5050 50  0000 C CNN
@@
 Connection ~ 4750 3800
 $Comp
-L SW_DIP_x01 SW?
+L SW_DIP_x01 SW1
 U 1 1 5997975E
 P 5050 1850
-F 0 "SW?" H 5050 2000 50  0000 C CNN
+F 0 "SW1" H 5050 2000 50  0000 C CNN
 F 1 "SW_DIP_x01" H 5050 1700 50  0000 C CNN
 F 2 "" H 5050 1850 50  0000 C CNN
@@
 $EndComp
 $Comp
-L SW_DIP_x01 SW?
+L SW_DIP_x01 SW2
 U 1 1 59979863
 P 6100 1850
-F 0 "SW?" H 6100 2000 50  0000 C CNN
+F 0 "SW2" H 6100 2000 50  0000 C CNN
 F 1 "SW_DIP_x01" H 6100 1700 50  0000 C CNN
 F 2 "" H 6100 1850 50  0000 C CNN
@@
 	7050 1850 6350 1850
 Connection ~ 7050 3500
+Wire Wire Line
+	3700 3400 3700 4700
+Text Label 3750 4700 0    60   ~ 0
+GND
+Text GLabel 3600 4700 0    60   Input ~ 0
+GND
+Wire Wire Line
+	3600 4700 3750 4700
+Connection ~ 3700 4700
+Text GLabel 5550 1650 0    60   Input ~ 0
+GND
+Wire Wire Line
+	5550 1650 5550 1850
+Connection ~ 5550 1850
+Text GLabel 3550 1900 0    60   Input ~ 0
+3.7vBAT
+$Comp
+L R 100k
+U 1 1 59A72962
+P 3850 1900
+F 0 "100k" V 3930 1900 50  0000 C CNN
+F 1 "R" V 3850 1900 50  0000 C CNN
+F 2 "" V 3780 1900 50  0000 C CNN
+F 3 "" H 3850 1900 50  0000 C CNN
+	1    3850 1900
+	0    1    1    0
+$EndComp
+Wire Wire Line
+	3550 1900 3700 1900
+Wire Wire Line
+	4100 3200 4900 3200
+$Comp
+L R R?
+U 1 1 59A73ABA
+P 4100 2150
+F 0 "R?" V 4180 2150 50  0000 C CNN
+F 1 "R" V 4100 2150 50  0000 C CNN
+F 2 "" V 4030 2150 50  0000 C CNN
+F 3 "" H 4100 2150 50  0000 C CNN
+	1    4100 2150
+	1    0    0    -1
+$EndComp
+Wire Wire Line
+	4100 3200 4100 2300
+Wire Wire Line
+	4100 2000 4100 1900
+Wire Wire Line
+	4100 1900 4000 1900
 $EndSCHEMATC
